Commit message: support python3

File: parkingdemo_description/urdf/fusion_13_structure.urdf.xacro (robot description, xacro)
@@ -119,10 +119,10 @@
       </collision>
     </link>
-    <joint name="base_link" type="fixed">
+    <joint name="base_link_joint" type="fixed">
       <origin xyz="0 0 0.33" rpy="0 0 0"/>
       <parent link="base_footprint"/>
       <child link="base_link"/>
     </joint>
-    <joint name="steer_fl" type="continuous">
+    <joint name="steer_fl_joint" type="continuous">
       <origin xyz="2.85 0.79121 0" rpy="0 0 0"/>
       <parent link="base_link"/>
@@ -131,5 +131,5 @@
      <!-- <limit lower="-0.65" upper="0.65" effort="0" velocity="0"/> -->
     </joint>
-    <joint name="steer_fr" type="continuous">
+    <joint name="steer_fr_joint" type="continuous">
       <origin xyz="2.85 -0.79121 0" rpy="0 0 0"/>
       <parent link="base_link"/>
@@ -138,5 +138,5 @@
      <!-- <limit lower="-0.65" upper="0.65" effort="0" velocity="0"/> -->
     </joint>
-    <joint name="wheel_fl" type="continuous">
+    <joint name="wheel_fl_joint" type="continuous">
       <origin xyz="0 0 0" rpy="1.570796 0 -3.141593"/>
       <parent link="steer_fl"/>
@@ -145,5 +145,5 @@
       <limit effort="0" velocity="22.0"/>
     </joint>
-    <joint name="wheel_fr" type="continuous">
+    <joint name="wheel_fr_joint" type="continuous">
       <origin xyz="0 0 0" rpy="1.570796 0 -3.141593"/>
       <parent link="steer_fr"/>
@@ -152,5 +152,5 @@
       <limit effort="0" velocity="22.0"/>
     </joint>
-    <joint name="wheel_rl" type="continuous">
+    <joint name="wheel_rl_joint" type="continuous">
       <origin xyz="0 0.7874 0" rpy="1.570796 0 -3.141593"/>
       <parent link="base_link"/>
@@ -159,5 +159,5 @@
       <limit effort="5000.0" velocity="22.0"/>
     </joint>
-    <joint name="wheel_rr" type="continuous">
+    <joint name="wheel_rr_joint" type="continuous">
       <origin xyz="0 -0.7874 0" rpy="1.570796 0 -3.141593"/>
       <parent link="base_link"/>
@@ -169,5 +169,5 @@
   <transmission name="tran1">
     <type>transmission_interface/SimpleTransmission</type>
-    <joint name="wheel_rr">
+    <joint name="wheel_rr_joint">
       <hardwareInterface>hardware_interface/EffortJointInterface</hardwareInterface>
     </joint>
@@ -179,5 +179,5 @@
   <transmission name="tran2">
     <type>transmission_interface/SimpleTransmission</type>
-    <joint name="wheel_rl">
+    <joint name="wheel_rl_joint">
       <hardwareInterface>hardware_interface/EffortJointInterface</hardwareInterface>
     </joint>
@@ -189,5 +189,5 @@
   <transmission name="tran3">
     <type>transmission_interface/SimpleTransmission</type>
-    <joint name="wheel_fr">
+    <joint name="wheel_fr_joint">
       <hardwareInterface>hardware_interface/EffortJointInterface</hardwareInterface>
     </joint>
@@ -199,5 +199,5 @@
   <transmission name="tran4">
     <type>transmission_interface/SimpleTransmission</type>
-    <joint name="wheel_fl">
+    <joint name="wheel_fl_joint">
       <hardwareInterface>hardware_interface/EffortJointInterface</hardwareInterface>
     </joint>
@@ -209,5 +209,5 @@
   <transmission name="tran5">
     <type>transmission_interface/SimpleTransmission</type>
-    <joint name="steer_fr">
+    <joint name="steer_fr_joint">
       <hardwareInterface>hardware_interface/EffortJointInterface</hardwareInterface>
     </joint>
@@ -219,5 +219,5 @@
   <transmission name="tran6">
     <type>transmission_interface/SimpleTransmission</type>
-    <joint name="steer_fl">
+    <joint name="steer_fl_joint">
       <hardwareInterface>hardware_interface/EffortJointInterface</hardwareInterface>
     </joint>
@@ -232,5 +232,5 @@
       <alwaysOn>true</alwaysOn>
       <updateRate>50.0</updateRate>
-      <bodyName>base_link</bodyName>
+      <bodyName>base_footprint</bodyName>
       <topicName>ground_truth/state</topicName>
       <gaussianNoise>0.01</gaussianNoise>
